Commit message: Update URDF to include more joints

File: tesbot_description/urdf/tesbot.urdf (robot description, URDF)
Before this commit: robot tesbot, 5 links, 4 joints
Links:
- added link dump_end
- added link ladder_end
Joints:
- added joint dump: type prismatic, parent base_link, child dump_end, limit upper=0.20 effort=90 velocity=1000
- added joint ladder: type prismatic, parent base_link, child ladder_end, limit upper=0.20 effort=90 velocity=1000

Commit message: Fix joint locations

File: tesbot_description/urdf/tesbot.urdf (robot description, URDF)
Before this commit: robot tesbot, 7 links, 6 joints
Joints:
- joint base_to_left_back_wheel: origin xyz=-.3302 -.40005 0 -> xyz=-.2667 -.365125 0
- joint base_to_left_front_wheel: origin xyz=-.338836 .40005 0 -> xyz=-.2667 .365125 0
- joint base_to_right_back_wheel: origin xyz=.3302 -.40005 0 -> xyz=.2667 -.365125 0
- joint base_to_right_front_wheel: origin xyz=.338836 .40005 0 -> xyz=.2667 .365125 0
